Commit message: Same fingertips with Allegro

File: assets/leap_hand/robot.urdf (robot description, URDF)
Before this commit: robot onshape, 17 links, 16 joints
Links:
- link fingertip: mass 0.016 -> 0.0168; geometry collision sphere radius=0.01235; visual mesh filename=fingertip.stl
- link fingertip_2: mass 0.016 -> 0.0168; geometry collision sphere radius=0.01235; visual mesh filename=fingertip.stl
- link fingertip_3: mass 0.016 -> 0.0168; geometry collision sphere radius=0.01235; visual mesh filename=fingertip.stl
- link thumb_fingertip: mass 0.049 -> 0.0168; geometry collision sphere radius=0.01235; visual mesh filename=thumb_fingertip.stl

Commit message: Remove fingertip mesh visual from LEAP URDF, keep sphere only
The original fingertip.stl mesh visual was redundant since we use
sphere collision geometry for physics. Keeping only the sphere
visual makes the collision geometry clearly visible during debugging.

File: assets/leap_hand/robot.urdf (robot description, URDF)
Before this commit: robot onshape, 17 links, 16 joints
Links:
- link fingertip: geometry collision sphere radius=0.01235; visual sphere radius=0.01235
- link fingertip_2: geometry collision sphere radius=0.01235; visual sphere radius=0.01235
- link fingertip_3: geometry collision sphere radius=0.01235; visual sphere radius=0.01235
- link thumb_fingertip: geometry collision sphere radius=0.01235; visual sphere radius=0.01235
